File: ecad/SATA0.sch (KiCad schematic (older format))
At the start: 57 parts, among them IC12 TUSB9261IPVP, IC13 IS25LQ010B, J15 Conn_SATA, Y4 40MHz

Commit message: Fixing Schematic Annotation
Other:
- note added: "This schematic follows roughly the reccommendations \ngiven in the TUSB9261 Implementation Guide\nhttps://www.ti.com/lit/pdf/slla315"
- note removed: "This schematic follows roughly the reccommendations \ngiven in the TUSB9262 Implementation Guide\nhttps://www.ti.com/lit/pdf/slla315"
Changed lines of the file:
@@
 $EndComp
 Text Notes 5650 6350 0    50   ~ 0
-This schematic follows roughly the reccommendations \ngiven in the TUSB9262 Implementation Guide\nhttps://www.ti.com/lit/pdf/slla315
+This schematic follows roughly the reccommendations \ngiven in the TUSB9261 Implementation Guide\nhttps://www.ti.com/lit/pdf/slla315
 $EndSCHEMATC
